File: usb4x1mux.brd (EAGLE design)
At the start: 123 x 80 mm, 44 parts, among them IC10 SN74LVC1G139DCTR, IC3 LDO5-3.3-SOT23, U1 LPC812M101JDH16

Commit message: move git tag mark
Parts:
- moved GIT1 60.9 mm to (68.9, 65.8)
Changed lines of the file:
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@@
 </autorouter>
 <elements>
-<element name="GIT1" library="git-revision" package="GIT-REVISION_1.7" value="" x="35.6" y="14.8" smashed="yes">
-<attribute name="NOT_COMPONENT" value="YES" x="35.6" y="14.8" size="1.778" layer="27" display="off"/>
-<attribute name="VALUE" x="35.6" y="14.8" size="1.7" layer="21" ratio="12" align="center"/>
+<element name="GIT1" library="git-revision" package="GIT-REVISION_1.7" value="" x="68.9" y="65.8" smashed="yes">
+<attribute name="NOT_COMPONENT" value="YES" x="68.9" y="65.8" size="1.778" layer="27" display="off"/>
+<attribute name="VALUE" x="68.9" y="65.8" size="1.7" layer="21" ratio="12" align="center"/>
 </element>
 <element name="PCB1" library="mylib" package="HAMMOND-1593K" value="" x="32.7" y="11.7" smashed="yes"/>

Commit message: update library; move git hash tag silk
Parts:
- moved GIT1 0.81 mm to (69.0, 65.0)
Changed lines of the file:
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@@
 </autorouter>
 <elements>
-<element name="GIT1" library="git-revision" package="GIT-REVISION_1.7" value="" x="68.9" y="65.8" smashed="yes">
-<attribute name="NOT_COMPONENT" value="YES" x="68.9" y="65.8" size="1.778" layer="27" display="off"/>
-<attribute name="VALUE" x="68.9" y="65.8" size="1.7" layer="21" ratio="12" align="center"/>
+<element name="GIT1" library="git-revision" package="GIT-REVISION_1.7" value="" x="69" y="65" smashed="yes">
+<attribute name="NOT_COMPONENT" value="YES" x="69" y="65" size="1.778" layer="27" display="off"/>
+<attribute name="VALUE" x="69" y="65" size="1.7" layer="21" ratio="12" align="center"/>
 </element>
 <element name="PCB1" library="mylib" package="HAMMOND-1593K" value="" x="32.7" y="11.7" smashed="yes"/>
@@
 <element name="CON7" library="mylib" package="PH127-2X5MG-1.5" value="" x="112.3" y="40" smashed="yes" rot="MR180">
 <attribute name="NAME" x="115.9" y="38.3" size="1" layer="26" ratio="20" rot="MR90"/>
+<attribute name="AKIZUKI" value="C-10904" x="112.3" y="40" size="1.778" layer="28" rot="MR180" display="off"/>
 </element>
 <element name="SW5" library="mylib" package="SW-TACTSW-2P" value="" x="62.2" y="17.5" smashed="yes" rot="R90">
@@
 <element name="U1" library="mylib" package="SOT65P510X450X110-16N" value="LPC812M101JDH16" x="55.7" y="28" smashed="yes">
 <attribute name="DIGIKEY" value="568-10436-5-ND" x="50.5" y="28" size="1.778" layer="27" display="off"/>
-<attribute name="SMD_PAD" value="16" x="50.5" y="28" size="1.778" layer="27" display="off"/>
 <attribute name="NAME" x="51.9" y="30.7" size="1.27" layer="25" font="vector" ratio="17" align="center"/>
 <attribute name="VALUE" x="55.7" y="28" size="1.27" layer="27" font="vector" ratio="17" align="center"/>
+<attribute name="SMD-PAD" value="16" x="55.7" y="28" size="1.778" layer="27" display="off"/>
 </element>
 <element name="C13" library="mylib" package="CR-1608" value="0.1u/1005" x="56" y="32.7" smashed="yes">
@@
 <element name="CON8" library="mylib" package="PH127-2X5MG-1.5" value="" x="67.7" y="28" smashed="yes" rot="R270">
 <attribute name="NAME" x="66.1" y="31.5" size="1" layer="25" ratio="20"/>
+<attribute name="AKIZUKI" value="C-10904" x="67.7" y="28" size="1.778" layer="27" rot="R270" display="off"/>
 </element>
 <element name="IC10" library="mylib" package="SOT65P315X290-8N" value="SN74LVC1G139DCTR" x="61.7" y="28.4" smashed="yes">
